Commit message: d435 incorporated in simulation

File: turtlebot3_description/urdf/turtlebot3_waffle.gazebo.xacro (robot description, xacro)
@@ -55,5 +55,5 @@
     <plugin name="turtlebot3_waffle_controller" filename="libgazebo_ros_diff_drive.so">
       <commandTopic>cmd_vel</commandTopic>
-      <odometryTopic>acl_jackal/jackal_velocity_controller/odom</odometryTopic>
+      <odometryTopic>odom</odometryTopic>
       <odometryFrame>odom</odometryFrame>
       <odometrySource>world</odometrySource>
@@ -75,13 +75,12 @@
   </gazebo>
   <gazebo>
-    <!-- <gravity>0 0 -9.81</gravity> -->
     <plugin name="imu_plugin" filename="libgazebo_ros_imu.so">
       <alwaysOn>true</alwaysOn>
       <bodyName>imu_link</bodyName>
       <frameName>imu_link</frameName>
-      <topicName>acl_jackal/forward/imu</topicName>
+      <topicName>imu</topicName>
       <serviceName>imu_service</serviceName>
       <gaussianNoise>0.0</gaussianNoise>
-      <updateRate>400</updateRate>
+      <updateRate>0</updateRate>
       <imu>
         <noise>
@@ -89,12 +88,12 @@
           <rate>
             <mean>0.0</mean>
-            <stddev>1e-4</stddev>
-            <bias_mean>0.0</bias_mean>
-            <bias_stddev>1e-2</bias_stddev>
+            <stddev>2e-4</stddev>
+            <bias_mean>0.0000075</bias_mean>
+            <bias_stddev>0.0000008</bias_stddev>
           </rate>
           <accel>
             <mean>0.0</mean>
             <stddev>1.7e-2</stddev>
-            <bias_mean>0.0</bias_mean>
+            <bias_mean>0.1</bias_mean>
             <bias_stddev>0.001</bias_stddev>
           </accel>
@@ -179,143 +178,3 @@
     </sensor>
   </gazebo> -->
-  <!-- D455  https://github.com/pal-robotics-forks/realsense/blob/melodic-devel/realsense2_description/urdf/_d455.gazebo.xacro -->
-  <!-- Load parameters to model's main link-->
-  <xacro:property name="deg_to_rad" value="0.01745329251994329577" />
-  <xacro:property name="reference_link" value="camera_link" />
-  <xacro:property name="camera_name" value="camera" />
-  <xacro:property name="topics_ns" value="camera" />
-  <xacro:property name="depth_optical_frame" value="camera_depth_optical_frame" />
-  <xacro:property name="color_optical_frame" value="camera_rgb_optical_frame" />
-  <xacro:property name="infrared1_optical_frame" value="camera_infra1_optical_frame" />
-  <xacro:property name="infrared2_optical_frame" value="camera_infra2_optical_frame" />
-  <xacro:property name="publish_pointcloud" value="true" />
-  <gazebo reference="${reference_link}">
-    <self_collide>0</self_collide>
-    <enable_wind>0</enable_wind>
-    <kinematic>0</kinematic>
-    <gravity>1</gravity>
-    <!--<mu>1</mu>-->
-    <mu2>1</mu2>
-    <fdir1>0 0 0</fdir1>
-    <!--<slip1>0</slip1>
-    <slip2>0</slip2>-->
-    <kp>1e+13</kp>
-    <kd>1</kd>
-    <!--<max_vel>0.01</max_vel>
-    <min_depth>0</min_depth>-->
-    <sensor name="${camera_name}color" type="camera">
-      <camera name="${camera_name}">
-        <horizontal_fov>${87*deg_to_rad}</horizontal_fov>
-        <image>
-          <width>640</width>
-          <height>480</height>
-          <format>RGB_INT8</format>
-        </image>
-        <clip>
-          <near>0.1</near>
-          <far>100</far>
-        </clip>
-        <noise>
-          <type>gaussian</type>
-          <mean>0.0</mean>
-          <stddev>0.007</stddev>
-        </noise>
-      </camera>
-      <always_on>1</always_on>
-      <update_rate>30</update_rate>
-      <visualize>1</visualize>
-    </sensor>
-    <sensor name="${camera_name}ired1" type="camera">
-      <camera name="${camera_name}">
-        <horizontal_fov>${87*deg_to_rad}</horizontal_fov>
-        <image>
-          <width>640</width>
-          <height>480</height>
-          <format>L_INT8</format>
-        </image>
-        <clip>
-          <near>0.1</near>
-          <far>100</far>
-        </clip>
-        <noise>
-          <type>gaussian</type>
-          <mean>0.0</mean>
-          <stddev>0.05</stddev>
-        </noise>
-      </camera>
-      <always_on>1</always_on>
-      <update_rate>20</update_rate>
-      <visualize>0</visualize>
-    </sensor>
-    <sensor name="${camera_name}ired2" type="camera">
-      <camera name="${camera_name}">
-        <horizontal_fov>${87*deg_to_rad}</horizontal_fov>
-        <image>
-          <width>640</width>
-          <height>480</height>
-          <format>L_INT8</format>
-        </image>
-        <clip>
-          <near>0.1</near>
-          <far>100</far>
-        </clip>
-        <noise>
-          <type>gaussian</type>
-          <mean>0.0</mean>
-          <stddev>0.05</stddev>
-        </noise>
-      </camera>
-      <always_on>1</always_on>
-      <update_rate>20</update_rate>
-      <visualize>0</visualize>
-    </sensor>
-    <sensor name="${camera_name}depth" type="depth">
-      <camera name="${camera_name}">
-        <horizontal_fov>${87*deg_to_rad}</horizontal_fov>
-        <image>
-          <width>640</width>
-          <height>480</height>
-        </image>
-        <clip>
-          <near>0.1</near>
-          <far>100</far>
-        </clip>
-        <noise>
-          <type>gaussian</type>
-          <mean>0.0</mean>
-          <stddev>0.100</stddev>
-        </noise>
-      </camera>
-      <always_on>1</always_on>
-      <update_rate>90</update_rate>
-      <visualize>0</visualize>
-    </sensor>
-  </gazebo>
-  <gazebo>
-    <!-- <plugin name="${topics_ns}" filename="librealsense_gazebo_plugin.so"> -->
-    <plugin name="acl_jackal/forward" filename="librealsense_gazebo_plugin.so">
-      <prefix>${camera_name}</prefix>
-      <depthUpdateRate>30.0</depthUpdateRate>
-      <colorUpdateRate>30.0</colorUpdateRate>
-      <infraredUpdateRate>30.0</infraredUpdateRate>
-      <depthTopicName>depth/image_rect_raw</depthTopicName>
-      <depthCameraInfoTopicName>depth/camera_info</depthCameraInfoTopicName>
-      <colorTopicName>color/image_raw</colorTopicName>
-      <colorCameraInfoTopicName>color/camera_info</colorCameraInfoTopicName>
-      <infrared1TopicName>infra1/image_rect_raw</infrared1TopicName>
-      <infrared1CameraInfoTopicName>infra1/camera_info</infrared1CameraInfoTopicName>
-      <infrared2TopicName>infra2/image_rect_raw</infrared2TopicName>
-      <infrared2CameraInfoTopicName>infra2/camera_info</infrared2CameraInfoTopicName>
-      <colorOpticalframeName>${color_optical_frame}</colorOpticalframeName>
-      <depthOpticalframeName>${depth_optical_frame}</depthOpticalframeName>
-      <infrared1OpticalframeName>${infrared1_optical_frame}</infrared1OpticalframeName>
-      <infrared2OpticalframeName>${infrared2_optical_frame}</infrared2OpticalframeName>
-      <rangeMinDepth>0.520</rangeMinDepth>
-      <rangeMaxDepth>10.0</rangeMaxDepth>
-      <pointCloud>${publish_pointcloud}</pointCloud>
-      <pointCloudTopicName>depth/color/points</pointCloudTopicName>
-      <pointCloudCutoff>0.25</pointCloudCutoff>
-      <pointCloudCutoffMax>9.0</pointCloudCutoffMax>
-    </plugin>
-  </gazebo>
 </robot>

File: turtlebot3_description/urdf/turtlebot3_waffle.urdf.xacro (robot description, xacro)
@@ -3,4 +3,5 @@
   <xacro:include filename="$(find turtlebot3_description)/urdf/common_properties.xacro"/>
   <xacro:include filename="$(find turtlebot3_description)/urdf/turtlebot3_waffle.gazebo.xacro"/>
+  <xacro:include filename="$(find realsense2_description)/urdf/_d435.urdf.xacro" />
   <xacro:property name="r200_cam_rgb_px" value="0.005"/>
   <xacro:property name="r200_cam_rgb_py" value="0.018"/>
@@ -35,4 +36,13 @@
     </inertial>
   </link>
+  <joint name="d435_camera_joint" type="fixed">
+    <parent link="base_link"/>
+    <child link="d435_camera_link" />
+    <origin xyz="0.1 0 0.1" rpy="0 0 0"/>
+  </joint>
+  <link name="d435_camera_link" />
+  <xacro:sensor_d435 parent="d435_camera_link" name="camera" use_nominal_extrinsics="true" add_plug="true" use_mesh="true">
+      <origin xyz="0 0 0" rpy="0 0 0"/>
+  </xacro:sensor_d435>
   <joint name="wheel_left_joint" type="continuous">
     <parent link="base_link"/>
@@ -164,224 +174,3 @@
     </inertial>
   </link>
-  <joint name="camera_joint" type="fixed">
-    <origin xyz="0.064 -0.065 0.094" rpy="0 0 0"/>
-    <parent link="base_link"/>
-    <child link="camera_link"/>
-  </joint>
-  <link name="camera_link">
-    <visual>
-     <origin xyz="0 0 0" rpy="1.57 0 1.57"/>
-      <geometry>
-       <mesh filename="package://turtlebot3_description/meshes/sensors/r200.dae" />
-      </geometry>
-    </visual>
-    <collision>
-      <origin xyz="0.003 0.065 0.007" rpy="0 0 0"/>
-      <geometry>
-        <box size="0.012 0.132 0.020"/>
-      </geometry>
-    </collision>
-    <!-- This inertial field needs doesn't contain reliable data!! -->
-<!--   <inertial>
-      <mass value="0.564" />
-      <origin xyz="0 0 0" />
-      <inertia ixx="0.003881243" ixy="0.0" ixz="0.0"
-               iyy="0.000498940" iyz="0.0"
-               izz="0.003879257" />
-    </inertial>-->
-  </link>
-  <joint name="camera_rgb_joint" type="fixed">
-    <origin xyz="${r200_cam_rgb_px} ${r200_cam_rgb_py} ${r200_cam_rgb_pz}" rpy="0 0 0"/>
-    <parent link="camera_link"/>
-    <child link="camera_rgb_frame"/>
-  </joint>
-  <link name="camera_rgb_frame"/>
-  <joint name="camera_rgb_optical_joint" type="fixed">
-    <origin xyz="0 0 0" rpy="-1.57 0 -1.57"/>
-    <parent link="camera_rgb_frame"/>
-    <child link="camera_rgb_optical_frame"/>
-  </joint>
-  <link name="camera_rgb_optical_frame"/>
-  <joint name="camera_depth_joint" type="fixed">
-    <origin xyz="${r200_cam_rgb_px} ${r200_cam_rgb_py + r200_cam_depth_offset} ${r200_cam_rgb_pz}" rpy="0 0 0"/>
-    <parent link="camera_link"/>
-    <child link="camera_depth_frame"/>
-  </joint>
-  <link name="camera_depth_frame"/>
-  <joint name="camera_depth_optical_joint" type="fixed">
-    <origin xyz="0 0 0" rpy="-1.57 0 -1.57"/>
-    <parent link="camera_depth_frame"/>
-    <child link="camera_depth_optical_frame"/>
-  </joint>
-  <link name="camera_depth_optical_frame"/>
-  <xacro:include filename="$(find turtlebot3_description)/urdf/_d455.gazebo.xacro"/>
-  <xacro:include filename="$(find turtlebot3_description)/urdf/_usb_plug.urdf.xacro" />
-  <xacro:macro name="sensor_d455" params="parent *origin name:=camera topics_ns:=camera use_nominal_extrinsics:=true add_plug:=false use_mesh:=true publish_pointcloud:=true">
-    <xacro:property name="M_PI" value="3.1415926535897931" />
-    <!-- The following values are approximate, and the camera node
-     publishing TF values with actual calibrated camera extrinsic values -->
-    <xacro:property name="d455_cam_depth_to_infra1_offset" value="0.0"/>
-    <xacro:property name="d455_cam_depth_to_infra2_offset" value="-0.095"/>
-    <xacro:property name="d455_cam_depth_to_color_offset" value="-0.059"/>
-    <!-- The following values model the aluminum peripherial case for the
-  	d455 camera, with the camera joint represented by the actual
-  	peripherial camera tripod mount -->
-    <xacro:property name="d455_cam_width" value="0.124"/>
-    <xacro:property name="d455_cam_height" value="0.029"/>
-    <xacro:property name="d455_cam_depth" value="0.026"/>
-    <xacro:property name="d455_cam_mount_from_center_offset" value="0.0158"/>
-    <!-- glass cover is 0.1 mm inwards from front aluminium plate -->
-    <xacro:property name="d455_glass_to_front" value="0.1e-3"/>
-    <!-- see datasheet Revision 009, Fig. 4-4 page 68 -->
-    <xacro:property name="d455_zero_depth_to_glass" value="4.55e-3"/>
-    <!-- convenience precomputation to avoid clutter-->
-    <xacro:property name="d455_mesh_x_offset" value="${d455_cam_mount_from_center_offset-d455_glass_to_front-d455_zero_depth_to_glass}"/>
-    <!-- The following offset is relative to the physical d455 camera peripherial
-  	camera tripod mount -->
-    <xacro:property name="d455_cam_depth_px" value="${d455_cam_mount_from_center_offset}"/>
-    <xacro:property name="d455_cam_depth_py" value="0.0475"/>
-    <xacro:property name="d455_cam_depth_pz" value="${d455_cam_height/2}"/>
-    <material name="${name}_aluminum">
-    <color rgba="0.5 0.5 0.5 1"/>
-    </material>
-    <!-- camera body, with origin at bottom screw mount -->
-    <joint name="${name}_joint" type="fixed">
-      <xacro:insert_block name="origin" />
-      <parent link="${parent}"/>
-      <child link="${name}_bottom_screw_frame" />
-    </joint>
-    <link name="${name}_bottom_screw_frame"/>
-    <joint name="${name}_link_joint" type="fixed">
-      <origin xyz="${d455_mesh_x_offset} ${d455_cam_depth_py} ${d455_cam_depth_pz}" rpy="0 0 0"/>
-      <parent link="${name}_bottom_screw_frame"/>
-      <child link="${name}_link" />
-    </joint>
-    <link name="${name}_link">
-      <visual>
-        <xacro:if value="${use_mesh}">
-          <!-- the mesh origin is at front plate in between the two infrared camera axes -->
-          <origin xyz="${d455_zero_depth_to_glass + d455_glass_to_front} ${-d455_cam_depth_py} 0" rpy="${M_PI/2} 0 ${M_PI/2}"/>
-          <geometry>
-            <mesh filename="package://realsense2_description/meshes/d455.stl" scale="0.001 0.001 0.001" />
-          </geometry>
-        </xacro:if>
-        <xacro:unless value="${use_mesh}">
-          <origin xyz="${d455_zero_depth_to_glass-d455_cam_depth/2} ${-d455_cam_depth_py} 0" rpy="0 0 0"/>
-          <geometry>
-            <box size="${d455_cam_depth} ${d455_cam_width} ${d455_cam_height}"/>
-          </geometry>
-          <material name="${name}_aluminum"/>
-        </xacro:unless>
-      </visual>
-      <collision>
-        <origin xyz="${d455_zero_depth_to_glass-d455_cam_depth/2} ${-d455_cam_depth_py} 0" rpy="0 0 0"/>
-        <geometry>
-          <box size="${d455_cam_depth} ${d455_cam_width} ${d455_cam_height}"/>
-        </geometry>
-      </collision>
-      <inertial>
-        <!-- The following are not reliable values, and should not be used for modeling -->
-        <mass value="0.072" />
-        <origin xyz="0 0 0" />
-        <inertia ixx="0.003881243" ixy="0.0" ixz="0.0" iyy="0.000498940" iyz="0.0" izz="0.003879257" />
-      </inertial>
-    </link>
-    <!-- Use the nominal extrinsics between camera frames if the calibrated extrinsics aren't being published. e.g. running the device in simulation  -->
-    <xacro:if value="${use_nominal_extrinsics}">
-      <!-- camera depth joints and links -->
-      <joint name="${name}_depth_joint" type="fixed">
-        <origin xyz="0 0 0" rpy="0 0 0"/>
-        <parent link="${name}_link"/>
-        <child link="${name}_depth_frame" />
-      </joint>
-      <link name="${name}_depth_frame"/>
-      <joint name="${name}_depth_optical_joint" type="fixed">
-        <origin xyz="0 0 0" rpy="${-M_PI/2} 0 ${-M_PI/2}" />
-        <parent link="${name}_depth_frame" />
-        <child link="${name}_depth_optical_frame" />
-      </joint>
-      <link name="${name}_depth_optical_frame"/>
-      <!-- camera left IR joints and links -->
-      <joint name="${name}_infra1_joint" type="fixed">
-        <origin xyz="0 ${d455_cam_depth_to_infra1_offset} 0" rpy="0 0 0" />
-        <parent link="${name}_link" />
-        <child link="${name}_infra1_frame" />
-      </joint>
-      <link name="${name}_infra1_frame"/>
-      <joint name="${name}_infra1_optical_joint" type="fixed">
-        <origin xyz="0 0 0" rpy="${-M_PI/2} 0 ${-M_PI/2}" />
-        <parent link="${name}_infra1_frame" />
-        <child link="${name}_infra1_optical_frame" />
-      </joint>
-      <link name="${name}_infra1_optical_frame"/>
-      <!-- camera right IR joints and links -->
-      <joint name="${name}_infra2_joint" type="fixed">
-        <origin xyz="0 ${d455_cam_depth_to_infra2_offset} 0" rpy="0 0 0" />
-        <parent link="${name}_link" />
-        <child link="${name}_infra2_frame" />
-      </joint>
-      <link name="${name}_infra2_frame"/>
-      <joint name="${name}_infra2_optical_joint" type="fixed">
-        <origin xyz="0 0 0" rpy="${-M_PI/2} 0 ${-M_PI/2}" />
-        <parent link="${name}_infra2_frame" />
-        <child link="${name}_infra2_optical_frame" />
-      </joint>
-      <link name="${name}_infra2_optical_frame"/>
-      <!-- camera color joints and links -->
-      <joint name="${name}_color_joint" type="fixed">
-        <origin xyz="0 ${d455_cam_depth_to_color_offset} 0" rpy="0 0 0" />
-        <parent link="${name}_link" />
-        <child link="${name}_color_frame" />
-      </joint>
-      <link name="${name}_color_frame"/>
-      <joint name="${name}_color_optical_joint" type="fixed">
-        <origin xyz="0 0 0" rpy="${-M_PI/2} 0 ${-M_PI/2}" />
-        <parent link="${name}_color_frame" />
-        <child link="${name}_color_optical_frame" />
-      </joint>
-      <link name="${name}_color_optical_frame"/>
-      <!-- IMU -->
-      <!-- see datasheet Revision 009, page 114 -->
-      <xacro:property name="d455_imu_px" value="-0.01602"/>
-      <xacro:property name="d455_imu_py" value="-0.03022"/>
-      <xacro:property name="d455_imu_pz" value="+0.0074"/>
-      <link name="${name}_accel_frame" />
-      <link name="${name}_accel_optical_frame" />
-      <link name="${name}_gyro_frame" />
-      <link name="${name}_gyro_optical_frame" />
-      <link name="${name}_imu_optical_frame" />
-      <joint name="${name}_accel_joint" type="fixed">
-        <origin xyz = "${d455_imu_px} ${d455_imu_py} ${d455_imu_pz}" rpy = "0 0 0" />
-        <parent link="${name}_link" />
-        <child link="${name}_accel_frame" />
-      </joint>
-      <joint name="${name}_accel_optical_joint" type="fixed">
-        <origin xyz = "0 0 0" rpy = "${-M_PI/2} 0 ${-M_PI/2}" />
-        <parent link="${name}_accel_frame" />
-        <child link="${name}_accel_optical_frame" />
-      </joint>
-      <joint name="${name}_gyro_joint" type="fixed">
-        <origin xyz = "${d455_imu_px} ${d455_imu_py} ${d455_imu_pz}" rpy = "0 0 0" />
-        <parent link="${name}_link" />
-        <child link="${name}_gyro_frame" />
-      </joint>
-      <joint name="${name}_gyro_optical_joint" type="fixed">
-        <origin xyz = "0 0 0" rpy = "${-M_PI/2} 0 ${-M_PI/2}" />
-        <parent link="${name}_gyro_frame" />
-        <child link="${name}_gyro_optical_frame" />
-      </joint>
-      <joint name="${name}_imu_optical_joint" type="fixed">
-        <origin xyz = "0 0 0" rpy = "0 0 0" />
-        <parent link="${name}_gyro_optical_frame" />
-        <child link="${name}_imu_optical_frame" />
-      </joint>
-    </xacro:if>
-    <xacro:if value="${add_plug}">
-      <xacro:usb_plug parent="${name}_link" name="${name}_usb_plug">
-        <origin xyz="${-0.00406-d455_cam_depth_px} ${-0.03701-d455_cam_depth_py} ${-d455_cam_depth_pz}" rpy="${M_PI/2} 0 0"/>
-      </xacro:usb_plug>
-    </xacro:if>
-    <!-- Realsense Gazebo Plugin -->
-    <xacro:gazebo_d455 camera_name="${name}" reference_link="${name}_link" topics_ns="${topics_ns}" depth_optical_frame="${name}_depth_optical_frame" color_optical_frame="${name}_color_optical_frame" infrared1_optical_frame="${name}_infra1_ir_optical_frame" infrared2_optical_frame="${name}_infra2_ir_optical_frame" publish_pointcloud="${publish_pointcloud}"/>
-  </xacro:macro>
 </robot>
